Commit message: Serielle Kommunikation zu Arduino Mega läuft

File: urdf/imars_lite.urdf (robot description, URDF)
Before this commit: robot imars_lite, 7 links, 6 joints
Links:
- removed link base_footprint
- added link robot_footprint
Joints:
- removed joint base_joint
- added joint footprint_joint: type fixed, parent base_link, child robot_footprint, origin xyz=0.0 0.0 ${-base_height-0.17} rpy=0 0 0
- joint depth_camera_joint: origin xyz=${camera_xoff} ${camera_yoff} ${camera_zoff} rpy=0 ${-0*pi/180} 0 -> xyz=${camera_xoff} ${camera_yoff} ${camera_zoff} rpy=0 ${15*pi/180} 0

Commit message: Serial_interface_function receive added

File: urdf/imars_lite.urdf (robot description, URDF)
Before this commit: robot imars_lite, 7 links, 6 joints
Joints:
- joint depth_camera_joint: parent head_link -> base_link
